File: 2350/hardware/WEACT-RP2350B/1.0/msx-picoverse.kicad_pcb (KiCad board)
At the start: 2 copper layers, 0 parts

Commit message: My first cartridge
Parts:
- added C1: 0.1uF, Capacitor_SMD:C_0603_1608Metric_Pad1.08x0.95mm_HandSolder, F.Cu at (46.9, 69.0)
- added C12: 4.7uF, Capacitor_SMD:C_0603_1608Metric_Pad1.08x0.95mm_HandSolder, F.Cu at (46.6, 64.0)
- added C14: 1nF, Capacitor_SMD:C_0603_1608Metric_Pad1.08x0.95mm_HandSolder, F.Cu at (42.1, 64.0)
- added C17: 1nF, Capacitor_SMD:C_0603_1608Metric_Pad1.08x0.95mm_HandSolder, F.Cu at (37.6, 64.0)
- added C18: 1uF, Capacitor_SMD:C_0603_1608Metric_Pad1.08x0.95mm_HandSolder, F.Cu at (37.6, 60.9)
- added C19: 100nF, Capacitor_SMD:C_0603_1608Metric_Pad1.08x0.95mm_HandSolder, F.Cu at (37.6, 57.8)
- added C2: 10uF, Capacitor_SMD:C_0603_1608Metric_Pad1.08x0.95mm_HandSolder, F.Cu at (52.9, 69.0)
- added C20: 4.7uF, Capacitor_SMD:C_0603_1608Metric_Pad1.08x0.95mm_HandSolder, F.Cu at (37.9, 53.0)
- added D1: 1N5819, Diode_SMD:D_SOD-123, F.Cu at (53.0, 59.7)
- added EDG1: MSX_CON, libraries:msx-con-MSXCART, F.Cu at (86.2, 72.2)
- added J2: Micro_SD_Card, Connector_Card:microSD_HC_Molex_47219-2001, F.Cu at (126.9, 66.2)
- added JP1: Jumper_2_Open, Jumper:SolderJumper-2_P1.3mm_Open_RoundedPad1.0x1.5mm, F.Cu at (67.9, 51.2)
- added R1: 2K, Resistor_SMD:R_0603_1608Metric_Pad0.98x0.95mm_HandSolder, F.Cu at (129.4, 91.6)
- added R10: 10K, Resistor_SMD:R_0603_1608Metric_Pad0.98x0.95mm_HandSolder, F.Cu at (42.2, 52.9)
- added R2: 10K, Resistor_SMD:R_0603_1608Metric_Pad0.98x0.95mm_HandSolder, F.Cu at (129.4, 95.6)
- added R3: 10K, Resistor_SMD:R_0603_1608Metric_Pad0.98x0.95mm_HandSolder, F.Cu at (124.4, 95.8)
- added R4: 10K, Resistor_SMD:R_0603_1608Metric_Pad0.98x0.95mm_HandSolder, F.Cu at (124.4, 87.5)
- added R5: 10K, Resistor_SMD:R_0603_1608Metric_Pad0.98x0.95mm_HandSolder, F.Cu at (129.3, 87.5)
- added R6: 10K, Resistor_SMD:R_0603_1608Metric_Pad0.98x0.95mm_HandSolder, F.Cu at (124.4, 91.6)
- added R7: 10K, Resistor_SMD:R_0603_1608Metric_Pad0.98x0.95mm_HandSolder, F.Cu at (37.7, 69.0)
- added R9: 10K, Resistor_SMD:R_0603_1608Metric_Pad0.98x0.95mm_HandSolder, F.Cu at (42.4, 69.0)
- added U2: MCP6001-OT, Package_TO_SOT_SMD:SOT-23-5, F.Cu at (45.6, 58.7)
- added U3: ~, WEACT_RP2350b:WeAct_RP2350B_headers, F.Cu at (93.3, 68.8)
Routing:
- net GND: track 0.00 -> 206.0 mm, vias 0 -> 8
- net +5V: track 0.00 -> 162.2 mm
- net PI_SOUND: track 0.00 -> 85.3 mm, vias 0 -> 2
- net RESET: track 0.00 -> 83.3 mm, vias 0 -> 3
- net BUSDIR: track 0.00 -> 82.7 mm, vias 0 -> 6
- net WAIT: track 0.00 -> 71.3 mm, vias 0 -> 2
- net A9: track 0.00 -> 69.5 mm, vias 0 -> 1
- net A0: track 0.00 -> 67.3 mm
- net A2: track 0.00 -> 65.3 mm
- net A6: track 0.00 -> 64.9 mm, vias 0 -> 2
- net A7: track 0.00 -> 64.5 mm, vias 0 -> 3
- net Net-(D1-A): track 0.00 -> 64.1 mm, vias 0 -> 1
- net A4: track 0.00 -> 64.1 mm
- net A11: track 0.00 -> 61.9 mm, vias 0 -> 1
- net A8: track 0.00 -> 61.9 mm, vias 0 -> 2
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Other:
- board outline added: 100.1 x 64.6 mm
- board text added: "PicoVerse Plus With SCC V1.0"

Commit message: v1.1 error in print
Routing:
- net RESET: track 83.3 -> 78.6 mm, vias 3 -> 4
Changed lines of the file:
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@@
+	)
+	(segment
+		(start 105.9688 95.885)
+		(end 105.9434 95.8596)
+		(width 0.25)
+		(layer "F.Cu")
+		(net 13)
 	)
 	(segment
@@
 	)
 	(segment
+		(start 111.379 95.885)
+		(end 105.9688 95.885)
+		(width 0.25)
+		(layer "F.Cu")
+		(net 13)
+	)
+	(segment
 		(start 113.538 95.758)
 		(end 123.524 95.758)
@@
 	)
 	(via
+		(at 105.9434 95.8596)
+		(size 0.6)
+		(drill 0.3)
+		(layers "F.Cu" "B.Cu")
+		(net 13)
+	)
+	(via
 		(at 111.379 95.885)
 		(size 0.5)
@@
 	)
 	(segment
-		(start 113.538 95.758)
-		(end 113.538 97.282)
-		(width 0.2)
-		(layer "B.Cu")
-		(net 13)
-	)
-	(segment
-		(start 113.538 97.282)
-		(end 106.196 104.624)
-		(width 0.2)
-		(layer "B.Cu")
-		(net 13)
-	)
-	(segment
-		(start 106.196 113.111)
-		(end 104.324 113.111)
-		(width 0.2)
+		(start 105.9434 100.5332)
+		(end 102.7176 103.759)
+		(width 0.25)
 		(layer "B.Cu")
 		(net 13)
@@
 	)
 	(segment
+		(start 102.7176 103.759)
+		(end 102.72 103.7614)
+		(width 0.25)
+		(layer "B.Cu")
+		(net 13)
+	)
+	(segment
 		(start 113.665 58.674)
 		(end 112.301 60.038)
@@
 	)
 	(segment
-		(start 106.196 104.624)
-		(end 106.196 113.111)
-		(width 0.2)
-		(layer "B.Cu")
-		(net 13)
-	)
-	(segment
-		(start 104.324 113.111)
-		(end 102.72 111.507)
-		(width 0.2)
-		(layer "B.Cu")
-		(net 13)
-	)
-	(segment
 		(start 113.411 95.885)
 		(end 113.538 95.758)
@@
 	)
 	(segment
+		(start 105.9434 95.8596)
+		(end 105.9434 100.5332)
+		(width 0.25)
+		(layer "B.Cu")
+		(net 13)
+	)
+	(segment
+		(start 102.72 103.7614)
+		(end 102.72 109)
+		(width 0.25)
+		(layer "B.Cu")
+		(net 13)
+	)
+	(segment
 		(start 114.816 98.809)
 		(end 114.816 85.225)
@@
 	)
 	(segment
-		(start 105.26 95.019)
+		(start 106.6546 103.3272)
+		(end 106.6546 93.6244)
+		(width 0.25)
+		(layer "B.Cu")
+		(net 18)
+	)
+	(segment
+		(start 106.6546 93.6244)
 		(end 113.665 86.614)
 		(width 0.25)
@@
 	(segment
 		(start 105.26 109)
-		(end 105.26 95.019)
+		(end 105.26 104.7218)
+		(width 0.25)
+		(layer "B.Cu")
+		(net 18)
+	)
+	(segment
+		(start 105.26 104.7218)
+		(end 106.6546 103.3272)
 		(width 0.25)
 		(layer "B.Cu")
@@
 	)
 	(segment
+		(start 105.2068 108.9468)
+		(end 105.2068 91.1678)
+		(width 0.2)
+		(layer "F.Cu")
+		(net 27)
+	)
+	(segment
 		(start 87.884 86.614)
 		(end 78.105 86.614)
@@
 	)
 	(segment
-		(start 105.26 91.221)
-		(end 100.78 86.741)
-		(width 0.2)
-		(layer "F.Cu")
-		(net 27)
-	)
-	(segment
 		(start 105.26 109)
 		(end 105.26 104.879)
@@
 	)
 	(segment
+		(start 105.2068 91.1678)
+		(end 100.78 86.741)
+		(width 0.2)
+		(layer "F.Cu")
+		(net 27)
+	)
+	(segment
 		(start 105.26 109)
-		(end 105.26 91.221)
-		(width 0.2)
-		(layer "F.Cu")
+		(end 105.2068 108.9468)
+		(width 0.2)
+		(layer "F.Cu")
